File: pcb01/pcb01.kicad_pcb (KiCad board)
At the start: 2 copper layers, 118.1 x 98.4 mm, 36 parts, among them J1 DIN41612_02x32_AC, J10 Conn_01x02_Socket, J2 Data Bus, J3 Address Bus, J4 Display, J5 UART, J6 UART_IRQ, J7 Jmp_Irq, J8 Jmp_NMI, J9 Ram1 Enable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

Commit message: small update
Parts:
- X1: footprint Package_DIP:DIP-14_W7.62mm_Socket -> Package_DIP:DIP-14_W7.62mm
Changed lines of the file:
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@@
     )
   )
-  (footprint "Package_DIP:DIP-14_W7.62mm_Socket" (layer "F.Cu")
+  (footprint "Package_DIP:DIP-14_W7.62mm" (layer "F.Cu")
     (at 26.67 64.77)
-    (descr "14-lead though-hole mounted DIP package, row spacing 7.62 mm (300 mils), Socket")
-    (tags "THT DIP DIL PDIP 2.54mm 7.62mm 300mil Socket")
+    (descr "14-lead though-hole mounted DIP package, row spacing 7.62 mm (300 mils)")
+    (tags "THT DIP DIL PDIP 2.54mm 7.62mm 300mil")
     (property "Sheetfile" "pcb01.kicad_sch")
     (property "Sheetname" "")
@@
         (effects (font (size 1 1) (thickness 0.15)))
     )
-    (fp_line (start -1.33 -1.39) (end -1.33 16.63)
-      (stroke (width 0.12) (type solid)) (layer "F.SilkS"))
-    (fp_line (start -1.33 16.63) (end 8.95 16.63)
-      (stroke (width 0.12) (type solid)) (layer "F.SilkS"))
     (fp_line (start 1.16 -1.33) (end 1.16 16.57)
       (stroke (width 0.12) (type solid)) (layer "F.SilkS"))
@@
     (fp_line (start 6.46 16.57) (end 6.46 -1.33)
       (stroke (width 0.12) (type solid)) (layer "F.SilkS"))
-    (fp_line (start 8.95 -1.39) (end -1.33 -1.39)
-      (stroke (width 0.12) (type solid)) (layer "F.SilkS"))
-    (fp_line (start 8.95 16.63) (end 8.95 -1.39)
-      (stroke (width 0.12) (type solid)) (layer "F.SilkS"))
     (fp_arc (start 4.81 -1.33) (mid 3.81 -0.33) (end 2.81 -1.33)
       (stroke (width 0.12) (type solid)) (layer "F.SilkS"))
-    (fp_line (start -1.55 -1.6) (end -1.55 16.85)
+    (fp_line (start -1.1 -1.55) (end -1.1 16.8)
       (stroke (width 0.05) (type solid)) (layer "F.CrtYd"))
-    (fp_line (start -1.55 16.85) (end 9.15 16.85)
+    (fp_line (start -1.1 16.8) (end 8.7 16.8)
       (stroke (width 0.05) (type solid)) (layer "F.CrtYd"))
-    (fp_line (start 9.15 -1.6) (end -1.55 -1.6)
+    (fp_line (start 8.7 -1.55) (end -1.1 -1.55)
       (stroke (width 0.05) (type solid)) (layer "F.CrtYd"))
-    (fp_line (start 9.15 16.85) (end 9.15 -1.6)
+    (fp_line (start 8.7 16.8) (end 8.7 -1.55)
       (stroke (width 0.05) (type solid)) (layer "F.CrtYd"))
-    (fp_line (start -1.27 -1.33) (end -1.27 16.57)
-      (stroke (width 0.1) (type solid)) (layer "F.Fab"))
-    (fp_line (start -1.27 16.57) (end 8.89 16.57)
-      (stroke (width 0.1) (type solid)) (layer "F.Fab"))
     (fp_line (start 0.635 -0.27) (end 1.635 -1.27)
       (stroke (width 0.1) (type solid)) (layer "F.Fab"))
@@
       (stroke (width 0.1) (type solid)) (layer "F.Fab"))
     (fp_line (start 6.985 16.51) (end 0.635 16.51)
-      (stroke (width 0.1) (type solid)) (layer "F.Fab"))
-    (fp_line (start 8.89 -1.33) (end -1.27 -1.33)
-      (stroke (width 0.1) (type solid)) (layer "F.Fab"))
-    (fp_line (start 8.89 16.57) (end 8.89 -1.33)
       (stroke (width 0.1) (type solid)) (layer "F.Fab"))
     (pad "1" thru_hole rect (at 0 0) (size 1.6 1.6) (drill 0.8) (layers "*.Cu" "*.Mask")
@@
     (pad "14" thru_hole oval (at 7.62 0) (size 1.6 1.6) (drill 0.8) (layers "*.Cu" "*.Mask")
       (net 2 "VCC") (pinfunction "Vcc") (pintype "power_in"))
-    (model "${KICAD6_3DMODEL_DIR}/Package_DIP.3dshapes/DIP-14_W7.62mm_Socket.wrl"
+    (model "${KICAD6_3DMODEL_DIR}/Package_DIP.3dshapes/DIP-14_W7.62mm.wrl"
       (offset (xyz 0 0 0))
       (scale (xyz 1 1 1))

Commit message: connect GPIO0
Parts:
- added J11: Conn_01x09, Connector_PinSocket_2.54mm:PinSocket_1x09_P2.54mm_Vertical, F.Cu at (106.0, 86.4)
- added RV1: R_Potentiometer_Small, Potentiometer_THT:Potentiometer_Vishay_T73YP_Vertical, F.Cu at (135.3, 111.1)
Connections:
- J1 pad a16: unconnected-(J1-Pin_a16-Pada16) -> /~{SYS_CLK}
- J4 pad 3: unconnected-(J4-Pin_3-Pad3) -> /LCD_BIAS
- U6 pad 12: unconnected-(U6-Q7-Pad12) -> Net-(J11-Pin_9)
- U6 pad 13: unconnected-(U6-Q6-Pad13) -> Net-(J11-Pin_8)
- U6 pad 14: unconnected-(U6-Q5-Pad14) -> Net-(J11-Pin_7)
- U6 pad 15: unconnected-(U6-Q4-Pad15) -> Net-(J11-Pin_6)
- U6 pad 16: unconnected-(U6-Q3-Pad16) -> Net-(J11-Pin_5)
- U6 pad 17: unconnected-(U6-Q2-Pad17) -> Net-(J11-Pin_4)
- U6 pad 18: unconnected-(U6-Q1-Pad18) -> Net-(J11-Pin_3)
- U6 pad 19: unconnected-(U6-Q0-Pad19) -> Net-(J11-Pin_2)
Routing:
- net /~{SYS_CLK}: track 0.00 -> 38.0 mm, vias 0 -> 3
- net /LCD_BIAS: track 0.00 -> 11.6 mm
- net Net-(J11-Pin_9): track 0.00 -> 3.81 mm
- net Net-(J11-Pin_8): track 0.00 -> 3.81 mm
- net Net-(J11-Pin_7): track 0.00 -> 3.81 mm
- net Net-(J11-Pin_6): track 0.00 -> 3.81 mm
- net Net-(J11-Pin_5): track 0.00 -> 3.81 mm
- net Net-(J11-Pin_4): track 0.00 -> 3.81 mm
- net Net-(J11-Pin_3): track 0.00 -> 3.81 mm
- net Net-(J11-Pin_2): track 0.00 -> 3.81 mm
- net /DISP_EN: track 115.7 -> 118.5 mm
