File: kicad/cpu_board_03/cpu_board_03.kicad_pcb (KiCad board)
At the start: 4 copper layers, 99.1 x 94.2 mm, 58 parts, among them J1 DIN41612_02x32_AC, J10 PLD_aux, J11 Conn_01x09, J6 Conn_01x02_Socket, J9 Ram1 Enable, SW1 SW_Reset, SW2 SW_PWR, U1 W65C02SxP, U10 74HC245, U11 74HC245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

Commit message: routing improvements
Parts:
- J10: footprint Connector_PinSocket_2.54mm:PinSocket_1x03_P2.54mm_Vertical -> Connector_PinHeader_2.54mm:PinHeader_1x03_P2.54mm_Vertical
Connections:
- net /~{SYS_CLK} renamed /~{PLD_O9}
- U10 pad 1: VCC -> GND
- U11 pad 1: VCC -> GND
- X1 pad 10: (no net) -> unconnected-(X1-NC-Pad10)
- X1 pad 12: (no net) -> unconnected-(X1-NC-Pad12)
- X1 pad 13: (no net) -> unconnected-(X1-NC-Pad13)
- X1 pad 2: (no net) -> unconnected-(X1-NC-Pad2)
- X1 pad 3: (no net) -> unconnected-(X1-NC-Pad3)
- X1 pad 4: (no net) -> unconnected-(X1-NC-Pad4)
- X1 pad 5: (no net) -> unconnected-(X1-NC-Pad5)
- X1 pad 6: (no net) -> unconnected-(X1-NC-Pad6)
- X1 pad 9: (no net) -> unconnected-(X1-NC-Pad9)
Routing:
- net GND: track 882.6 -> 927.3 mm, vias 23 -> 75
- net VCC: track 555.1 -> 533.0 mm
- net /SYS_CLK: track 131.2 -> 133.0 mm
- net /~{IO_RD_DIR}: track 62.7 -> 61.9 mm
- net /A6: track 125.9 -> 125.2 mm
- net /~{CS_ROM}: track 41.3 -> 41.9 mm
- net /A5: track 121.5 -> 120.9 mm
- net /A11: track 99.7 -> 99.2 mm
- net /GPIO00_O7: track 12.8 -> 12.3 mm
- net /GPIO00_O6: track 12.3 -> 11.8 mm
- net /GPIO00_O5: track 11.7 -> 11.2 mm
- net /GPIO00_O4: track 11.6 -> 11.1 mm
- net /GPIO00_O3: track 12.2 -> 11.7 mm
- net /GPIO00_O2: track 12.7 -> 12.2 mm
- net /GPIO00_O1: track 13.8 -> 13.3 mm
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Other:
- copper layers 4 -> 2
- board text added: "6502 SBC Mark3 'MI' cpu board 2025"
- board text added: "Addressbus"
- board text added: "Databus"
- board text added: "GND"
- board text added: "IO-Enable"
- board text added: "PLD I/O"
- board text added: "Reset/Irq"
- board text added: "VCC"
