File: kicad/cpu_board_03_4l/cpu_board_03_4l.kicad_sch (KiCad schematic)
At the start: 63 parts, among them J1 DIN41612_02x32_AC, J10 PLD_aux, J11 Conn_01x09, J6 Conn_01x02_Socket, J9 Ram1 Enable, SW1 SW_Reset, SW2 SW_PWR, U1 W65C02SxP, U10 74HC245, U11 74HC245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

Commit message: cleaned up pullup mess
Parts:
- removed D14: LED_Small, LED_SMD:LED_0805_2012Metric_Pad1.15x1.40mm_HandSolder, symbol Device:LED_Small
- removed R6, R7, R8: 10K, Resistor_SMD:R_0805_2012Metric_Pad1.20x1.40mm_HandSolder, symbol Device:R
- added U14: 74AHC1G04, Package_TO_SOT_SMD:SOT-23-5_HandSoldering, symbol 74xGxx:74AHC1G04
Connections:
- net CLOCK: now also U14.2
- net GND: now also J1.c29 (Pin_c29), U14.3 (GND)
- net VCC: now also J1.a29 (Pin_a29), U1.2 (RDY), U1.36 (BE), U14.5 (VCC)
- net ~{IO_WR}: no longer U13.1
- net ~{IRQ}: now also J1.c30 (Pin_c30); no longer J1.a29 (Pin_a29)
- net ~{NMI}: now also J1.a30 (Pin_a30); no longer J1.c30 (Pin_c30)
- removed net BE: J1.a30 (Pin_a30), U1.36 (BE)
- removed net RDY: J1.c29 (Pin_c29), U1.2 (RDY)
- new net: U13.1, U14.4
