File: kicad/vga_mem_output_01_4l/display_generator.kicad_sch (KiCad schematic)
At the start: 10 parts, among them U13 74LS163, U14 74LS163, U15 74LS163, U16 74LS163, U17 74LS163, U18 74LS163, U19 PAL20RS10, U20 PAL20RS10, U21 74LS08, Y1 CXO_DIP8

Commit message: routing fixes
Connections:
- net H0 renamed DG_PIXEL
Changed lines of the file:
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@@
+	(wire
+		(pts
+			(xy 71.12 24.13) (xy 64.77 24.13)
+		)
+		(stroke
+			(width 0)
+			(type default)
+		)
+	)
 	(wire
 		(pts
@@
 		(effects
 			(font
+				(size 1.27 1.27)
+			)
+			(justify left)
+		)
+	)
+	(hierarchical_label "DG_PIXEL"
+		(shape output)
+		(at 71.12 24.13 0)
+		(effects
+			(font
